Commit message: initial yam meshes drawn. URDF in progress

File: yam_description/yam.urdf (robot description, URDF)
Before this commit: robot yam, 11 links, 8 joints
Links:
- link camera_link: geometry collision cylinder length=0.0762 radius=0.0254; visual mesh filename=package://yam_description/meshes/visual/camera.stl scale=1.0 1.0 1.0
- link center_ultrasonic_link: geometry collision mesh filename=package://yam_description/meshes/collision/ultrasonic.stl scale=1.0 1.0 1.0; visual mesh filename=package://yam_description/meshes/visual/ultrasonic.stl scale=1.0 1.0 1.0
- link left_caster_wheel_link: geometry visual cylinder length=0.0254 radius=0.0127
- link left_drive_wheel_link: geometry visual cylinder length=0.01905 radius=0.0635
- link left_ultrasonic_link: geometry collision mesh filename=package://yam_description/meshes/collision/ultrasonic.stl scale=1.0 1.0 1.0; visual mesh filename=package://yam_description/meshes/visual/ultrasonic.stl scale=1.0 1.0 1.0
- link right_caster_wheel_link: geometry visual cylinder length=0.0254 radius=0.0127
- link right_drive_wheel_link: geometry visual cylinder length=0.01905 radius=0.0635
- link right_ultrasonic_link: geometry collision mesh filename=package://yam_description/meshes/collision/ultrasonic.stl scale=1.0 1.0 1.0; visual mesh filename=package://yam_description/meshes/visual/ultrasonic.stl scale=1.0 1.0 1.0
- link yam_body_link: geometry collision mesh filename=package://yam_description/meshes/collision/yam_body.stl scale=1.0 1.0 1.0; visual mesh filename=package://yam_description/meshes/visual/yam_body.stl scale=1.0 1.0 1.0
Joints:
- joint : origin xyz=0 0 0 -> xyz=0 0 0 rpy=0 0 0
- joint body_fixed_joint: origin xyz=0 0 0 -> xyz=0 0.0254 0 rpy=0 0 0
- joint camera_fixed_joint: origin xyz=0 0 0 -> xyz=0 0 0 rpy=0 0 0
- joint left_caster_wheel_fixed_joint: origin xyz=0 0 0 rpy=0 0 0 -> xyz=0.0889 -0.127 0 rpy=-1.57 0 0
- joint left_drive_wheel_joint: origin xyz=0 0 0 rpy=0 0 0 -> xyz=-0.0889 -0.127 0.0508 rpy=1.57 0 0
- joint left_ultrasonic_fixed_joint: origin xyz=0 0 0 -> xyz=0 0 0 rpy=0 0 0
- joint right_caster_wheel_fixed_joint: origin xyz=0 0 0 rpy=0 0 0 -> xyz=0.0889 0.127 0 rpy=1.57 0 0
- joint right_drive_wheel_joint: origin xyz=0 0 0 rpy=0 0 0 -> xyz=-0.0889 0.127 0.0508 rpy=-1.57 0 0
